Commit message: Corrected Basic P3AT defs

File: defs/robots/p3at/p3at.common.xacro (robot description, xacro)
@@ -2,5 +2,5 @@
 <robot xmlns:xacro="http://ros.org/wiki/xacro">
     <!-- Meshes -->
-    <xacro:property name="p3at_chasis_mesh" value="models/robots/p3at_meshes/chasis.stl" />
+    <xacro:property name="p3at_chasis_mesh" value="models/robots/p3at_meshes/chassis.stl" />
     <xacro:property name="p3at_wheel_mesh" value="models/robots/p3at_meshes/wheel.stl" />
     <xacro:property name="p3at_top_mesh" value="models/robots/p3at_meshes/top.stl" />

File: defs/robots/p3at/p3at.sdf.xacro (robot description, xacro)
@@ -127,10 +127,10 @@
         <wheelSeparation>0.4</wheelSeparation>
         <wheelDiameter>0.215</wheelDiameter>
-        <robotBaseFrame>base_link</robotBaseFrame>
+        <robotBaseFrame>${robot_name}/base_link</robotBaseFrame>
         <torque>200</torque>
         <!--MaxForce>5.0</MaxForce-->
         <commandTopic>cmd_vel</commandTopic>
         <odometryTopic>odom</odometryTopic>
-        <odometryFrame>odom</odometryFrame>
+        <odometryFrame>${robot_name}/odom</odometryFrame>
         <broadcastTF>1</broadcastTF>
     </plugin>

File: defs/robots/p3at/p3at.urdf.xacro (robot description, xacro)
@@ -6,17 +6,17 @@
 <xacro:macro name="p3at_chasis" >
     <!-- Chassis Links -->
-    <xacro:urdf_link _name="base_link" _xyz="0 0 0.177" _rpy="0 0 0"
+    <xacro:urdf_link_color _name="base_link" _xyz="0 0 0.177" _rpy="0 0 0"
         _mesh="${p3at_chasis_mesh}" _mass="10.0" _cg="0 0 0.177"
         _ixx="0.3338" _iyy="0.4783" _izz="0.3338" _ixy="0" _ixz="0" _iyz="0"
         _colorname="ChassisRed" _rgba="0.851 0.0 0.0 1.0" />
-    <xacro:urdf_link _name="top_plate" _xyz="0 0 0" _rpy="0 0 0"
+    <xacro:urdf_link_color _name="top_plate" _xyz="0 0 0" _rpy="0 0 0"
         _mesh="${p3at_top_mesh}" _mass="0.1" _cg="-0.025 0 -0.223"
         _ixx="1.0" _iyy="1.0" _izz="1.0" _ixy="0" _ixz="0" _iyz="0"
         _colorname="TopBlack" _rgba="0.038 0.038 0.038 1.0" />
-    <xacro:urdf_link _name="front_sonar" _xyz="0 0 0" _rpy="0 0 0"
+    <xacro:urdf_link_color _name="front_sonar" _xyz="0 0 0" _rpy="0 0 0"
         _mesh="${p3at_fsonar_mesh}" _mass="0.1" _cg="0 0 0"
         _ixx="1.0" _iyy="1.0" _izz="1.0" _ixy="0" _ixz="0" _iyz="0"
         _colorname="SonarYellow" _rgba="0.715 0.583 0.210 1.0" />
-    <xacro:urdf_link _name="back_sonar" _xyz="0 0 0" _rpy="0 0 0"
+    <xacro:urdf_link_color _name="back_sonar" _xyz="0 0 0" _rpy="0 0 0"
         _mesh="${p3at_bsonar_mesh}" _mass="0.1" _cg="0 0 0"
         _ixx="1.0" _iyy="1.0" _izz="1.0" _ixy="0" _ixz="0" _iyz="0"
@@ -34,5 +34,5 @@
 <!-- Front Axles + Wheels + Hubcaps -->
     <!-- Axle Front-->
-    <xacro:urdf_link _name="p3at_front_${suffix}_axle" _xyz="0 0 0" _rpy="0 0 0"
+    <xacro:urdf_link_color _name="p3at_front_${suffix}_axle" _xyz="0 0 0" _rpy="0 0 0"
         _mesh="${p3at_axle_mesh}" _mass="0.1" _cg="0 0 0"
         _ixx="1.0" _iyy="1.0" _izz="1.0" _ixy="0" _ixz="0" _iyz="0"
@@ -41,5 +41,5 @@
         _xyz="0.135 ${reflect*0.156} 0.111" _rpy="0 0 0" />
     <!-- Axle Back-->
-    <xacro:urdf_link _name="p3at_back_${suffix}_axle" _xyz="0 0 0" _rpy="0 0 0"
+    <xacro:urdf_link_color _name="p3at_back_${suffix}_axle" _xyz="0 0 0" _rpy="0 0 0"
         _mesh="${p3at_axle_mesh}" _mass="0.1" _cg="0 0 0"
         _ixx="1.0" _iyy="1.0" _izz="1.0" _ixy="0" _ixz="0" _iyz="0"
@@ -48,6 +48,6 @@
         _xyz="-0.134 ${reflect*0.156} 0.111" _rpy="0 0 0" />
 	<!-- Front Hub -->
-    <xacro:urdf_link _name="p3at_front_${suffix}_hub" _xyz="0 0 0" _rpy="0 0 0"
-        _mesh="${p3at_${suffix}_hubcap_mesh}" _mass="0.1" _cg="0 0 0"
+    <xacro:urdf_link_color _name="p3at_front_${suffix}_hub" _xyz="0 0 0" _rpy="0 0 0"
+        _mesh="models/robots/p3at_meshes/${suffix}_hubcap.stl" _mass="0.1" _cg="0 0 0"
         _ixx="1.0" _iyy="1.0" _izz="1.0" _ixy="0" _ixz="0" _iyz="0"
         _colorname="HubcapYellow" _rgba="1.0 0.811 0.151 1.0" />
@@ -55,6 +55,6 @@
         _xyz="0 ${reflect*0.041} 0" _rpy="0 0 0" />
     <!-- Back Hub -->
-    <xacro:urdf_link _name="p3at_back_${suffix}_hub" _xyz="0 0 0" _rpy="0 0 0"
-        _mesh="${p3at_${suffix}_hubcap_mesh}" _mass="0.1" _cg="0 0 0"
+    <xacro:urdf_link_color _name="p3at_back_${suffix}_hub" _xyz="0 0 0" _rpy="0 0 0"
+        _mesh="models/robots/p3at_meshes/${suffix}_hubcap.stl" _mass="0.1" _cg="0 0 0"
         _ixx="1.0" _iyy="1.0" _izz="1.0" _ixy="0" _ixz="0" _iyz="0"
         _colorname="HubcapYellow" _rgba="1.0 0.811 0.151 1.0" />
@@ -62,5 +62,5 @@
         _xyz="-0 ${reflect*0.041} 0" _rpy="0 0 0" />
     <!-- Front Wheel -->
-    <xacro:urdf_link _name="p3at_front_${suffix}_wheel" _xyz="0 0 0" _rpy="0 0 0"
+    <xacro:urdf_link_color _name="p3at_front_${suffix}_wheel" _xyz="0 0 0" _rpy="0 0 0"
         _mesh="${p3at_wheel_mesh}" _mass="0.5" _cg="0 0 0"
         _ixx="0.012411765597" _iyy="0.015218160428" _izz="0.011763977943" _ixy="0" _ixz="0" _iyz="0"
@@ -70,5 +70,5 @@
         _axis="0 1 0" _xyz="0 0 0" _rpy="0 0 0" _effort="100" _velocity="100" />
     <!-- Back Wheel -->
-    <xacro:urdf_link _name="p3at_back_${suffix}_wheel" _xyz="0 0 0" _rpy="0 0 0"
+    <xacro:urdf_link_color _name="p3at_back_${suffix}_wheel" _xyz="0 0 0" _rpy="0 0 0"
         _mesh="${p3at_wheel_mesh}" _mass="0.5" _cg="0 0 0"
         _ixx="0.012411765597" _iyy="0.015218160428" _izz="0.011763977943" _ixy="0" _ixz="0" _iyz="0"
