Commit message: Patched risewheelchair model

File: defs/robots/risewheelchair/risewheelchair.common.xacro (robot description, xacro)
@@ -1,16 +1,17 @@
 <?xml version="1.0"?>
 <robot xmlns:xacro="http://ros.org/wiki/xacro">
-<xacro:property name="wheelchair_base_mesh" value="models/robots/wheelchair1/Wheelchair_Structure.dae" />
-<xacro:property name="wheelchair_caster_mesh" value="models/robots/wheelchair1/Wheelchair_Caster.dae" />
-<xacro:property name="wheelchair_wheel_mesh" value="models/robots/wheelchair1/Wheelchair_Wheel.dae" />
-<xacro:property name="bender_body_mesh" value="models/robots/wheelchair1/Bender_Body.dae" />
-<xacro:property name="bender_head_mesh" value="models/robots/wheelchair1/Bender_Head.dae" />
+<xacro:property name="wheelchair_base_mesh" value="models/robots/risewheelchair/Wheelchair_Structure.dae" />
+<xacro:property name="wheelchair_caster_mesh" value="models/robots/risewheelchair/Wheelchair_Caster.dae" />
+<xacro:property name="wheelchair_wheel_mesh" value="models/robots/risewheelchair/Wheelchair_Wheel.dae" />
+<xacro:property name="bender_body_mesh" value="models/robots/risewheelchair/Bender_Body.dae" />
+<xacro:property name="bender_head_mesh" value="models/robots/risewheelchair/Bender_Head.dae" />
 <!-- Wheel Chair Data -->
-<xacro:property name="wheelchair_xyz" value="0 0 0" />
+<xacro:property name="wheelchair_z" value="0.1925" />
+<xacro:property name="wheelchair_xyz" value="0 0 ${wheelchair_z}" />
 <xacro:property name="wheelchair_rpy" value="0 0 0" />
 <xacro:property name="wheelchair_cg" value="0.2 0 0.2" />
 <xacro:property name="bender_x" value="0.106" />
 <xacro:property name="bender_y" value="0" />
-<xacro:property name="bender_z" value="0.508" />
+<xacro:property name="bender_z" value="${wheelchair_z + 0.508}" />
 <xacro:property name="bender_rpy" value="0 0 0" />
 <xacro:property name="bender_cg" value="0 0 0" />
@@ -24,6 +25,6 @@
 <xacro:property name="bender_head_gaz_xyz" value="${bender_x + bender_head_x} ${bender_y + bender_head_y} ${bender_z + bender_head_z}" />
 <!-- Wheel Data -->
-<xacro:property name="wheel_left_joint_xyz" value="0 0.2374 0"/>
-<xacro:property name="wheel_right_joint_xyz" value="0 -0.2374 0"/>
+<xacro:property name="wheel_left_joint_xyz" value="0 0.2374 ${wheelchair_z}"/>
+<xacro:property name="wheel_right_joint_xyz" value="0 -0.2374 ${wheelchair_z}"/>
 <xacro:property name="wheel_left_rpy" value="-1.57 0 0" />
 <xacro:property name="wheel_right_rpy" value="1.57 0 0" />
@@ -31,6 +32,6 @@
 <xacro:property name="wheel_axis" value="0 1 0" />
 <!-- Caster Wheel Data -->
-<xacro:property name="caster_left_joint_xyz" value="0.5203 0.2006 0.0376"/>
-<xacro:property name="caster_right_joint_xyz" value="0.5203 -0.2006 0.0376"/>
+<xacro:property name="caster_left_joint_xyz" value="0.5203 0.2006 ${wheelchair_z + 0.0376}"/>
+<xacro:property name="caster_right_joint_xyz" value="0.5203 -0.2006 ${wheelchair_z + 0.0376}"/>
 <xacro:property name="caster_left_rpy" value="0 0 0" />
 <xacro:property name="caster_right_rpy" value="0 0 0" />
@@ -87,5 +88,5 @@
 <xacro:property name="wheelchair_sicklms_x" value="0.8081" />
 <xacro:property name="wheelchair_sicklms_y" value="0" />
-<xacro:property name="wheelchair_sicklms_z" value="-0.01" />
+<xacro:property name="wheelchair_sicklms_z" value="${wheelchair_z -0.01}" />
 <xacro:property name="wheelchair_sicklms_z_visual_offset" value="0.0925" />
 <xacro:property name="wheelchair_sicklms_sensor_z_offset" value="0.063" />

File: defs/robots/risewheelchair/risewheelchair.sdf.xacro (robot description, xacro)
@@ -1,8 +1,8 @@
 ﻿<?xml version="1.0" ?>
 <sdf version="1.5" xmlns:xacro="http://www.ros.org/wiki/xacro">
-<xacro:include filename="$(find modeldb)/defs/robots/risewheelchair/risewheelchair.common.sdf.xacro" />
+<xacro:include filename="$(find riserobotdb)/defs/robots/risewheelchair/risewheelchair.common.sdf.xacro" />
 	<model name="risewheelchair">
 		<static>0</static>
-		<pose>0 0 1.2 0 0 0</pose>
+		<pose>0 0 0 0 0 0</pose>
 		<!-- Chassis -->
 			<link name="base_link">

Commit message: Wheelchair Stereo Camera

File: defs/robots/risewheelchair/risewheelchair.common.xacro (robot description, xacro)
@@ -92,6 +92,6 @@
 <xacro:property name="wheelchair_sicklms_sensor_z_offset" value="0.063" />
 <xacro:property name="wheelchair_sicklms_xyz" value="${wheelchair_sicklms_x} ${wheelchair_sicklms_y} ${wheelchair_sicklms_z}" />
-<xacro:property name="wheelchair_sicklms_frame" value="${wheelchair_sicklms_x} ${wheelchair_sicklms_y} ${wheelchair_sicklms_z + wheelchair_sicklms_z_visual_offset} 0 -0 1.5708" />
-<xacro:property name="wheelchair_sicklms_sensor" value="${wheelchair_sicklms_x} ${wheelchair_sicklms_y} ${wheelchair_sicklms_z + wheelchair_sicklms_sensor_z_offset} 0 0 0" />
+<xacro:property name="wheelchair_sicklms_frame" value="${wheelchair_sicklms_x} ${wheelchair_sicklms_y} ${wheelchair_sicklms_z_visual_offset -0.01} 0 -0 1.5708" />
+<xacro:property name="wheelchair_sicklms_sensor" value="${wheelchair_sicklms_x} ${wheelchair_sicklms_y} ${wheelchair_sicklms_sensor_z_offset -0.01} 0 0 0" />
 <!-- Camera in Simulation -->
 <xacro:property name="bender_eyes_xyz" value="0 0 0.1673" />

File: defs/robots/risewheelchair/risewheelchair.sdf.xacro (robot description, xacro)
@@ -2,4 +2,5 @@
 <sdf version="1.5" xmlns:xacro="http://www.ros.org/wiki/xacro">
 <xacro:include filename="$(find riserobotdb)/defs/robots/risewheelchair/risewheelchair.common.sdf.xacro" />
+<xacro:include filename="$(find riserobotdb)/defs/sensors/PTUD46MobileRanger/mobileranger_fixed.sdf.xacro" />
 	<model name="risewheelchair">
 		<static>0</static>
@@ -23,4 +24,7 @@
 				<xacro:sicklms200_laser robot_name="$(arg prefix)" id="0"
 					frame_pose="${wheelchair_sicklms_frame}" sensor_pose="${wheelchair_sicklms_sensor}"/>
+                <!-- Mobile Ranger Stereo Camera -->
+                <xacro:mobileranger_fixed robot_name="$(arg prefix)" _basepose="0.81 0.0 0.1755 0 0 0"
+                    left_pose="0.81 0.02921 0.25455 0 0 0" right_pose="0.81 -0.02921 0.25455 0 0 0"/>
 			</link>
 		<!-- Caster Wheels -->

File: defs/robots/risewheelchair/risewheelchair.urdf.xacro (robot description, xacro)
@@ -2,4 +2,5 @@
 <robot xmlns:xacro="http://ros.org/wiki/xacro" name="risewheelchair">
 <xacro:include filename="$(find riserobotdb)/defs/robots/risewheelchair/risewheelchair.common.urdf.xacro" />
+<xacro:include filename="$(find riserobotdb)/defs/sensors/PTUD46MobileRanger/mobileranger_fixed.urdf.xacro" />
 	<!-- Chassis -->
 	<xacro:urdf_link _name="base_link" _xyz="${wheelchair_xyz}" _rpy="${wheelchair_rpy}" _mesh="${wheelchair_base_mesh}"
@@ -17,4 +18,4 @@
 	</xacro:sicklms200_laser>
 	<!-- Mobile Ranger Stereo Camera -->
-	<!-- To ADD -->
+	<xacro:mobileranger_fixed _baselink="base_link" _basexyz="0.81 0.0 0.368" _baserpy="0 0 0" />
 </robot>
