Commit message: felis joint state publisher day end

File: defs/robots/felis/felis.common.xacro (robot description, xacro)
@@ -22,4 +22,7 @@
 <xacro:property name="felis_fulllink_centerlength" value="0.07" />
 <xacro:property name="felis_link_width" value="0.006" />
+<xacro:property name="joint_min_angle" value="0.087266463" />
+<!--xacro:property name="joint_min_angle" value="0" /-->
+<xacro:property name="joint_max_angle" value="3.124139361" />
 <!-- Base/Cage Data -->
 <xacro:property name="felis_xyz" value="0 0 ${felis_z}" />
@@ -45,5 +48,5 @@
 <xacro:property name="felis_linkA_joint_rr_rpy" value="-${angle_90d} ${felis_linkA_starting_angle} 0" />
 <!-- Link B Data -->
-<xacro:property name="felis_linkB_starting_angle" value="${angle_180d-angle_30d}" />
+<xacro:property name="felis_linkB_starting_angle" value="0" />
 <!-- Link C Data -->
 <!-- Link D Data -->
@@ -53,16 +56,16 @@
 <xacro:property name="spool_lower_angle" value="0" />
 <xacro:property name="spool_upper_angle" value="1.0" />
-<xacro:property name="quadleg_jointA_lower_angle"  value="0.0" />
-<xacro:property name="quadleg_jointA_upper_angle"  value="1.4" />
-<xacro:property name="quadleg_jointB_lower_angle"  value="0.0" />
-<xacro:property name="quadleg_jointB_upper_angle"  value="1.4" />
-<xacro:property name="quadleg_jointC_lower_angle"  value="0.0" />
-<xacro:property name="quadleg_jointC_upper_angle"  value="1.4" />
-<xacro:property name="quadleg_jointD_lower_angle"  value="0.0" />
-<xacro:property name="quadleg_jointD_upper_angle"  value="1.4" />
-<xacro:property name="quadleg_jointE_lower_angle"  value="0.0" />
-<xacro:property name="quadleg_jointE_upper_angle"  value="1.4" />
-<xacro:property name="quadleg_jointF_lower_angle"  value="0.0" />
-<xacro:property name="quadleg_jointF_upper_angle"  value="1.4" />
+<xacro:property name="quadleg_jointA_lower_angle"  value="-${joint_min_angle}" />
+<xacro:property name="quadleg_jointA_upper_angle"  value="-${joint_max_angle}" />
+<xacro:property name="quadleg_jointB_lower_angle"  value="${joint_min_angle}" />
+<xacro:property name="quadleg_jointB_upper_angle"  value="${joint_max_angle}" />
+<xacro:property name="quadleg_jointC_lower_angle"  value="${joint_min_angle}" />
+<xacro:property name="quadleg_jointC_upper_angle"  value="${joint_max_angle}" />
+<xacro:property name="quadleg_jointD_lower_angle"  value="-${joint_min_angle}" />
+<xacro:property name="quadleg_jointD_upper_angle"  value="-${joint_max_angle}" />
+<xacro:property name="quadleg_jointE_lower_angle"  value="-${joint_min_angle}" />
+<xacro:property name="quadleg_jointE_upper_angle"  value="-${joint_max_angle}" />
+<xacro:property name="quadleg_jointF_lower_angle"  value="${joint_min_angle}" />
+<xacro:property name="quadleg_jointF_upper_angle"  value="${joint_max_angle}" />
 <!-- Mass -->
 <xacro:property name="felis_baselink_mass" value="1.5" />

Commit message: Basic Joint constraints

File: defs/robots/felis/felis.common.xacro (robot description, xacro)
@@ -22,7 +22,6 @@
 <xacro:property name="felis_fulllink_centerlength" value="0.07" />
 <xacro:property name="felis_link_width" value="0.006" />
-<xacro:property name="joint_min_angle" value="0.087266463" />
-<!--xacro:property name="joint_min_angle" value="0" /-->
-<xacro:property name="joint_max_angle" value="3.124139361" />
+<xacro:property name="joint_min_angle" value="0.087266463" /><!-- Use Exact Values (For all links except A)-->
+<xacro:property name="joint_max_angle" value="3.124139361" /><!-- Use Exact Values (For all links except A)-->
 <!-- Base/Cage Data -->
 <xacro:property name="felis_xyz" value="0 0 ${felis_z}" />
@@ -38,5 +37,5 @@
 <xacro:property name="felis_spool_joint_rr_rpy" value="${angle_90d} -${angle_90d} 0" />
 <!-- Link A Data -->
-<xacro:property name="felis_linkA_starting_angle" value="${angle_180d-angle_15d}" />
+<xacro:property name="felis_linkA_starting_angle" value="0" />
 <xacro:property name="felis_linkA_joint_lf_xyz" value="${felis_jointfront_x+felis_motor_flipdifference} ${felis_jointfront_y} ${felis_leg_z}" />
 <xacro:property name="felis_linkA_joint_rf_xyz" value="${felis_jointfront_x+felis_motor_flipdifference} -${felis_jointfront_y} ${felis_leg_z}" />
@@ -56,16 +55,16 @@
 <xacro:property name="spool_lower_angle" value="0" />
 <xacro:property name="spool_upper_angle" value="1.0" />
-<xacro:property name="quadleg_jointA_lower_angle"  value="-${joint_min_angle}" />
-<xacro:property name="quadleg_jointA_upper_angle"  value="-${joint_max_angle}" />
-<xacro:property name="quadleg_jointB_lower_angle"  value="${joint_min_angle}" />
-<xacro:property name="quadleg_jointB_upper_angle"  value="${joint_max_angle}" />
-<xacro:property name="quadleg_jointC_lower_angle"  value="${joint_min_angle}" />
-<xacro:property name="quadleg_jointC_upper_angle"  value="${joint_max_angle}" />
-<xacro:property name="quadleg_jointD_lower_angle"  value="-${joint_min_angle}" />
-<xacro:property name="quadleg_jointD_upper_angle"  value="-${joint_max_angle}" />
-<xacro:property name="quadleg_jointE_lower_angle"  value="-${joint_min_angle}" />
-<xacro:property name="quadleg_jointE_upper_angle"  value="-${joint_max_angle}" />
-<xacro:property name="quadleg_jointF_lower_angle"  value="${joint_min_angle}" />
-<xacro:property name="quadleg_jointF_upper_angle"  value="${joint_max_angle}" />
+<xacro:property name="quadleg_jointA_lower_angle"  value="${angle_60d+angle_15d}" /> <!-- Use Exact Values -->
+<xacro:property name="quadleg_jointA_upper_angle"  value="${angle_180d - angle_15d}" /><!-- Use Exact Values -->
+<xacro:property name="quadleg_jointB_lower_angle"  value="${joint_min_angle}" /><!-- Use Exact Values -->
+<xacro:property name="quadleg_jointB_upper_angle"  value="${joint_max_angle}" /><!-- Use Exact Values -->
+<xacro:property name="quadleg_jointC_lower_angle"  value="${joint_min_angle}" /><!-- Use Exact Values -->
+<xacro:property name="quadleg_jointC_upper_angle"  value="${joint_max_angle}" /><!-- Use Exact Values -->
+<xacro:property name="quadleg_jointD_lower_angle"  value="-${joint_min_angle}" /><!-- Use Exact Values -->
+<xacro:property name="quadleg_jointD_upper_angle"  value="-${joint_max_angle}" /><!-- Use Exact Values -->
+<xacro:property name="quadleg_jointE_lower_angle"  value="-${joint_min_angle}" /><!-- Use Exact Values -->
+<xacro:property name="quadleg_jointE_upper_angle"  value="-${joint_max_angle}" /><!-- Use Exact Values -->
+<xacro:property name="quadleg_jointF_lower_angle"  value="${joint_min_angle}" /><!-- Use Exact Values -->
+<xacro:property name="quadleg_jointF_upper_angle"  value="${joint_max_angle}" /><!-- Use Exact Values -->
 <!-- Mass -->
 <xacro:property name="felis_baselink_mass" value="1.5" />
@@ -149,4 +148,5 @@
 <xacro:property name="angle_30d" value="0.523598776" />
 <xacro:property name="angle_45d" value="0.785398163" />
+<xacro:property name="angle_60d" value="1.047197551" />
 <xacro:property name="angle_90d" value="1.570796327" />
 <xacro:property name="angle_135d" value="2.35619449" />

Commit message: Felis CParam GUI Simple

File: defs/robots/felis/felis.common.xacro (robot description, xacro)
@@ -54,5 +54,5 @@
 <!-- Joints Constraints -->
 <xacro:property name="spool_lower_angle" value="0" />
-<xacro:property name="spool_upper_angle" value="1.0" />
+<xacro:property name="spool_upper_angle" value="${angle_60d}" />
 <xacro:property name="quadleg_jointA_lower_angle"  value="${angle_60d+angle_15d}" /> <!-- Use Exact Values -->
 <xacro:property name="quadleg_jointA_upper_angle"  value="${angle_180d - angle_15d}" /><!-- Use Exact Values -->

Commit message: Fixed urdf typo for rr_y

File: defs/robots/felis/felis.common.xacro (robot description, xacro)
@@ -55,5 +55,5 @@
 <xacro:property name="felis_linkA_joint_rf_xyz" value="${felis_linkA_joint_rf_x} ${felis_linkA_joint_rf_y} ${felis_linkA_joint_all_z}" />
 <xacro:property name="felis_linkA_joint_lr_xyz" value="${felis_linkA_joint_lr_x} ${felis_linkA_joint_lr_y} ${felis_linkA_joint_all_z}" />
-<xacro:property name="felis_linkA_joint_rr_xyz" value="${felis_linkA_joint_rr_x} ${felis_linkA_joint_lf_y} ${felis_linkA_joint_all_z}" />
+<xacro:property name="felis_linkA_joint_rr_xyz" value="${felis_linkA_joint_rr_x} ${felis_linkA_joint_rr_y} ${felis_linkA_joint_all_z}" />
 <xacro:property name="felis_linkA_joint_lf_rpy" value="${felis_linkA_joint_allrpy_r} ${felis_linkA_joint_allrpy_p} ${felis_linkA_joint_allrpy_y}" />
 <xacro:property name="felis_linkA_joint_rf_rpy" value="${felis_linkA_joint_allrpy_r} ${felis_linkA_joint_allrpy_p} ${felis_linkA_joint_allrpy_y}" />
