Commit message: Started setting up quadleg

File: defs/robots/felis/felis.common.urdf.xacro (robot description, xacro)
@@ -4,12 +4,29 @@
 <xacro:include filename="$(find riserobotdb)/defs/robots/felis/felis.common.xacro" />
 <!-- Leg Spool -->
-<xacro:macro name="rear_spool" params="suffix geom_rpy joint_xyz">
-	<xacro:urdf_link _name="${suffix}_rear_spool_link" _xyz="${felis_spool_xyz}" _rpy="${geom_rpy}"
+<xacro:macro name="spool" params="suffix portion geom_rpy joint_xyz">
+	<xacro:urdf_link _name="${suffix}_${portion}_spool_link" _xyz="${felis_spool_xyz}" _rpy="${geom_rpy}"
 		_mesh="${felis_spool_mesh}" _mass="${felis_spool_mass}" _cg="${felis_spool_cg}"
 		_ixx="${felis_spool_ixx}" _iyy="${felis_spool_iyy}" _izz="${felis_spool_izz}"
 		_ixy="${felis_spool_ixy}" _ixz="${felis_spool_ixz}" _iyz="${felis_spool_iyz}" />
-	<xacro:urdf_revolute_joint _name="${suffix}_rear_spool_joint" _parent="base_link"
-		_child="${suffix}_rear_spool_link" _axis="0 1 0" _xyz="${joint_xyz}" _rpy="0 0 0" _lower="${spool_lower_angle}"
+	<xacro:urdf_revolute_joint _name="${suffix}_${portion}_spool_joint" _parent="base_link"
+		_child="${suffix}_${portion}_spool_link" _axis="0 1 0" _xyz="${joint_xyz}" _rpy="0 0 0" _lower="${spool_lower_angle}"
 		_upper="${spool_upper_angle}" _effort="${spool_joint_effort}" _velocity="${spool_joint_velocity}" />
 </xacro:macro>
+<!-- Leg Link -->
+<xacro:macro name="quadleg" params="suffix portion geom_rpy joint_xyz">
+	<xacro:urdf_link _name="${suffix}_${portion}_quadleg_linkA" _xyz="${felis_linkA_xyz}" _rpy="${geom_rpy}"
+		_mesh="${felis_linkA_mesh}" _mass="${felis_linkA_mass}" _cg="${felis_linkA_cg}"
+		_ixx="${felis_linkA_ixx}" _iyy="${felis_linkA_iyy}" _izz="${felis_linkA_izz}"
+		_ixy="${felis_linkA_ixy}" _ixz="${felis_linkA_ixz}" _iyz="${felis_linkA_iyz}" />
+	<xacro:urdf_link _name="${suffix}_${portion}_quadleg_linkB" _xyz="${felis_linkB_xyz}" _rpy="${felis_linkB_rpy}"
+		_mesh="${felis_linkB_mesh}" _mass="${felis_linkB_mass}" _cg="${felis_linkB_cg}"
+		_ixx="${felis_linkB_ixx}" _iyy="${felis_linkB_iyy}" _izz="${felis_linkB_izz}"
+		_ixy="${felis_linkB_ixy}" _ixz="${felis_linkB_ixz}" _iyz="${felis_linkB_iyz}" />
+	<xacro:urdf_revolute_joint _name="${suffix}_${portion}_linkA_joint" _parent="base_link"
+		_child="${suffix}_${portion}_quadleg_linkA" _axis="0 1 0" _xyz="${joint_xyz}" _rpy="0 0 0" _lower="${quadleg_jointA_lower_angle}"
+		_upper="${quadleg_jointA_upper_angle}" _effort="${quadleg_joint_effort}" _velocity="${quadleg_joint_velocity}" />
+	<xacro:urdf_revolute_joint _name="${suffix}_${portion}_linkB_joint" _parent="${suffix}_${portion}_quadleg_linkA"
+		_child="${suffix}_${portion}_quadleg_linkB" _axis="0 1 0" _xyz="${felis_linkB_joint_xyz}" _rpy="0 0 0" _lower="${quadleg_jointB_lower_angle}"
+		_upper="${quadleg_jointB_upper_angle}" _effort="${quadleg_joint_effort}" _velocity="${quadleg_joint_velocity}" />
+</xacro:macro>
 </robot>

File: defs/robots/felis/felis.common.xacro (robot description, xacro)
@@ -4,10 +4,10 @@
 <xacro:property name="felis_base_mesh" value="models/robots/felis/felisbody.dae" />
 <xacro:property name="felis_spool_mesh" value="models/robots/felis/felislegspool.dae" />
-<xacro:property name="felis_linkA" value="models/robots/felis/felislinkA.dae" />
-<xacro:property name="felis_linkB" value="models/robots/felis/felislinkB.dae" />
-<xacro:property name="felis_linkC" value="models/robots/felis/felislinkC.dae" />
-<xacro:property name="felis_linkD" value="models/robots/felis/felislinkD.dae" />
-<xacro:property name="felis_linkE" value="models/robots/felis/felislinkE.dae" />
-<xacro:property name="felis_linkF" value="models/robots/felis/felislinkF.dae" />
+<xacro:property name="felis_linkA_mesh" value="models/robots/felis/felislinkA.dae" />
+<xacro:property name="felis_linkB_mesh" value="models/robots/felis/felislinkB.dae" />
+<xacro:property name="felis_linkC_mesh" value="models/robots/felis/felislinkC.dae" />
+<xacro:property name="felis_linkD_mesh" value="models/robots/felis/felislinkD.dae" />
+<xacro:property name="felis_linkE_mesh" value="models/robots/felis/felislinkE.dae" />
+<xacro:property name="felis_linkF_mesh" value="models/robots/felis/felislinkF.dae" />
 <!-- Base/Cage Data -->
 <xacro:property name="felis_z" value="0" />
@@ -18,17 +18,28 @@
 <xacro:property name="felis_spool_xyz" value="0 0 0" />
 <xacro:property name="felis_spool_cg" value="0 0 0" />
-<xacro:property name="felis_spool_jointA_xyz" value="-3 1 0" />
-<xacro:property name="felis_spool_jointA_rpy" value="0 3.14159 3.14159" />
-<xacro:property name="felis_spool_jointB_xyz" value="0 1 0" />
-<xacro:property name="felis_spool_jointC_xyz" value="0 1 0" />
-<xacro:property name="felis_spool_jointD_xyz" value="0 1 0" />
+<xacro:property name="felis_spool_joint1_xyz" value="-3 1 0" />
+<xacro:property name="felis_spool_joint1_rpy" value="0 3.14159 3.14159" />
+<xacro:property name="felis_spool_joint2_xyz" value="0 1 0" />
+<xacro:property name="felis_spool_joint2_rpy" value="0 3.14159 3.14159" />
+<xacro:property name="felis_spool_joint3_xyz" value="0 1 0" />
+<xacro:property name="felis_spool_joint3_rpy" value="0 3.14159 3.14159" />
+<xacro:property name="felis_spool_joint4_xyz" value="0 1 0" />
+<xacro:property name="felis_spool_joint4_rpy" value="0 3.14159 3.14159" />
 <!-- Link A Data -->
 <xacro:property name="felis_linkA_xyz" value="0 0 0" />
-<xacro:property name="felis_linkA_rpy" value="0 0 0" />
 <xacro:property name="felis_linkA_cg" value="0 0 0" />
+<xacro:property name="felis_linkA_joint1_xyz" value="-4 3 0" />
+<xacro:property name="felis_linkA_joint1_rpy" value="0 3.14159 3.14159" />
+<xacro:property name="felis_linkA_joint2_xyz" value="0 1 0" />
+<xacro:property name="felis_linkA_joint2_rpy" value="0 3.14159 3.14159" />
+<xacro:property name="felis_linkA_joint3_xyz" value="0 1 0" />
+<xacro:property name="felis_linkA_joint3_rpy" value="0 3.14159 3.14159" />
+<xacro:property name="felis_linkA_joint4_xyz" value="0 1 0" />
+<xacro:property name="felis_linkA_joint4_rpy" value="0 3.14159 3.14159" />
 <!-- Link B Data -->
 <xacro:property name="felis_linkB_xyz" value="0 0 0" />
 <xacro:property name="felis_linkB_rpy" value="0 0 0" />
 <xacro:property name="felis_linkB_cg" value="0 0 0" />
+<xacro:property name="felis_linkB_joint_xyz" value="1.5 0 0" />
 <!-- Link C Data -->
 <xacro:property name="felis_linkC_xyz" value="0 0 0" />
@@ -47,4 +58,11 @@
 <xacro:property name="felis_linkF_rpy" value="0 0 0" />
 <xacro:property name="felis_linkF_cg" value="0 0 0" />
+<!-- Joints Constraints -->
+<xacro:property name="spool_lower_angle" value="0" />
+<xacro:property name="spool_upper_angle" value="1.0" />
+<xacro:property name="quadleg_jointA_lower_angle"  value="0.0" />
+<xacro:property name="quadleg_jointA_upper_angle"  value="1.4" />
+<xacro:property name="quadleg_jointB_lower_angle"  value="0.0" />
+<xacro:property name="quadleg_jointB_upper_angle"  value="1.4" />
 <!-- Mass -->
 <xacro:property name="felis_baselink_mass" value="1.5" />
@@ -110,6 +128,6 @@
 <xacro:property name="spool_joint_effort" value="100" />
 <xacro:property name="spool_joint_velocity" value="50" />
-<xacro:property name="spool_lower_angle" value="0" />
-<xacro:property name="spool_upper_angle" value="1.0" />
+<xacro:property name="quadleg_joint_effort" value="100" />
+<xacro:property name="quadleg_joint_velocity" value="50" />
 <!-- SDF Specific parameters -->
 </robot>

File: defs/robots/felis/felis.urdf.xacro (robot description, xacro)
@@ -8,4 +8,6 @@
 	_ixy="${felis_baselink_ixy}" _ixz="${felis_baselink_ixz}" _iyz="${felis_baselink_iyz}"/>
 <!-- Spools -->
-<xacro:rear_spool suffix="left" geom_rpy="${felis_spool_jointA_rpy}" joint_xyz="${felis_spool_jointA_xyz}" />
+<xacro:spool suffix="left" portion="rear" geom_rpy="${felis_spool_joint1_rpy}" joint_xyz="${felis_spool_joint1_xyz}" />
+<!-- Legs -->
+<xacro:quadleg suffix="left" portion="front" geom_rpy="${felis_linkA_joint1_rpy}" joint_xyz="${felis_linkA_joint1_xyz}" />
 </robot>

Commit message: Fixed dae files for felis

File: defs/robots/felis/felis.common.urdf.xacro (robot description, xacro)
@@ -5,15 +5,15 @@
 <!-- Leg Spool -->
 <xacro:macro name="spool" params="suffix portion geom_rpy joint_xyz">
-	<xacro:urdf_link _name="${suffix}_${portion}_spool_link" _xyz="${felis_spool_xyz}" _rpy="${geom_rpy}"
+	<xacro:urdf_link _name="${suffix}_${portion}_spool_link" _xyz="${felis_spool_xyz}" _rpy="0 0 0"
 		_mesh="${felis_spool_mesh}" _mass="${felis_spool_mass}" _cg="${felis_spool_cg}"
 		_ixx="${felis_spool_ixx}" _iyy="${felis_spool_iyy}" _izz="${felis_spool_izz}"
 		_ixy="${felis_spool_ixy}" _ixz="${felis_spool_ixz}" _iyz="${felis_spool_iyz}" />
 	<xacro:urdf_revolute_joint _name="${suffix}_${portion}_spool_joint" _parent="base_link"
-		_child="${suffix}_${portion}_spool_link" _axis="0 1 0" _xyz="${joint_xyz}" _rpy="0 0 0" _lower="${spool_lower_angle}"
+		_child="${suffix}_${portion}_spool_link" _axis="0 0 1" _xyz="${joint_xyz}" _rpy="${geom_rpy}" _lower="${spool_lower_angle}"
 		_upper="${spool_upper_angle}" _effort="${spool_joint_effort}" _velocity="${spool_joint_velocity}" />
 </xacro:macro>
 <!-- Leg Link -->
 <xacro:macro name="quadleg" params="suffix portion geom_rpy joint_xyz">
-	<xacro:urdf_link _name="${suffix}_${portion}_quadleg_linkA" _xyz="${felis_linkA_xyz}" _rpy="${geom_rpy}"
+	<xacro:urdf_link _name="${suffix}_${portion}_quadleg_linkA" _xyz="${felis_linkA_xyz}" _rpy="0 0 0"
 		_mesh="${felis_linkA_mesh}" _mass="${felis_linkA_mass}" _cg="${felis_linkA_cg}"
 		_ixx="${felis_linkA_ixx}" _iyy="${felis_linkA_iyy}" _izz="${felis_linkA_izz}"
@@ -24,5 +24,5 @@
 		_ixy="${felis_linkB_ixy}" _ixz="${felis_linkB_ixz}" _iyz="${felis_linkB_iyz}" />
 	<xacro:urdf_revolute_joint _name="${suffix}_${portion}_linkA_joint" _parent="base_link"
-		_child="${suffix}_${portion}_quadleg_linkA" _axis="0 1 0" _xyz="${joint_xyz}" _rpy="0 0 0" _lower="${quadleg_jointA_lower_angle}"
+		_child="${suffix}_${portion}_quadleg_linkA" _axis="0 1 0" _xyz="${joint_xyz}" _rpy="${geom_rpy}" _lower="${quadleg_jointA_lower_angle}"
 		_upper="${quadleg_jointA_upper_angle}" _effort="${quadleg_joint_effort}" _velocity="${quadleg_joint_velocity}" />
 	<xacro:urdf_revolute_joint _name="${suffix}_${portion}_linkB_joint" _parent="${suffix}_${portion}_quadleg_linkA"

File: defs/robots/felis/felis.common.xacro (robot description, xacro)
@@ -13,22 +13,22 @@
 <xacro:property name="felis_z" value="0" />
 <xacro:property name="felis_xyz" value="0 0 ${felis_z}" />
-<xacro:property name="felis_rpy" value="0 0 3.14159" />
+<xacro:property name="felis_rpy" value="0 0 0" />
 <xacro:property name="felis_baselink_cg" value="0 0 0" />
 <!-- Spool Data -->
 <xacro:property name="felis_spool_xyz" value="0 0 0" />
 <xacro:property name="felis_spool_cg" value="0 0 0" />
-<xacro:property name="felis_spool_joint1_xyz" value="-3 1 0" />
-<xacro:property name="felis_spool_joint1_rpy" value="0 3.14159 3.14159" />
-<xacro:property name="felis_spool_joint2_xyz" value="0 1 0" />
-<xacro:property name="felis_spool_joint2_rpy" value="0 3.14159 3.14159" />
-<xacro:property name="felis_spool_joint3_xyz" value="0 1 0" />
-<xacro:property name="felis_spool_joint3_rpy" value="0 3.14159 3.14159" />
-<xacro:property name="felis_spool_joint4_xyz" value="0 1 0" />
-<xacro:property name="felis_spool_joint4_rpy" value="0 3.14159 3.14159" />
+<xacro:property name="felis_spool_joint1_xyz" value="0.04382 0.06030 0.02956" />
+<xacro:property name="felis_spool_joint1_rpy" value="-1.570796327 0 0" />
+<xacro:property name="felis_spool_joint2_xyz" value="0.04382 -0.06030 0.02956" />
+<xacro:property name="felis_spool_joint2_rpy" value="1.570796327 -1.570796327 0" />
+<xacro:property name="felis_spool_joint3_xyz" value="-0.12118 0.06840 0.02956" />
+<xacro:property name="felis_spool_joint3_rpy" value="-1.570796327 0 0" />
+<xacro:property name="felis_spool_joint4_xyz" value="-0.12118 -0.06840 0.02956" />
+<xacro:property name="felis_spool_joint4_rpy" value="1.570796327 -1.570796327 0" />
 <!-- Link A Data -->
 <xacro:property name="felis_linkA_xyz" value="0 0 0" />
 <xacro:property name="felis_linkA_cg" value="0 0 0" />
-<xacro:property name="felis_linkA_joint1_xyz" value="-4 3 0" />
-<xacro:property name="felis_linkA_joint1_rpy" value="0 3.14159 3.14159" />
+<xacro:property name="felis_linkA_joint1_xyz" value="0.06401 0.06030 0.00990" />
+<xacro:property name="felis_linkA_joint1_rpy" value="-1.570796327 2.35619449 0" />
 <xacro:property name="felis_linkA_joint2_xyz" value="0 1 0" />
 <xacro:property name="felis_linkA_joint2_rpy" value="0 3.14159 3.14159" />

File: defs/robots/felis/felis.urdf.xacro (robot description, xacro)
@@ -8,5 +8,8 @@
 	_ixy="${felis_baselink_ixy}" _ixz="${felis_baselink_ixz}" _iyz="${felis_baselink_iyz}"/>
 <!-- Spools -->
-<xacro:spool suffix="left" portion="rear" geom_rpy="${felis_spool_joint1_rpy}" joint_xyz="${felis_spool_joint1_xyz}" />
+<xacro:spool suffix="left" portion="front" geom_rpy="${felis_spool_joint1_rpy}" joint_xyz="${felis_spool_joint1_xyz}" />
+<xacro:spool suffix="right" portion="front" geom_rpy="${felis_spool_joint2_rpy}" joint_xyz="${felis_spool_joint2_xyz}" />
+<xacro:spool suffix="left" portion="rear" geom_rpy="${felis_spool_joint3_rpy}" joint_xyz="${felis_spool_joint3_xyz}" />
+<xacro:spool suffix="right" portion="rear" geom_rpy="${felis_spool_joint4_rpy}" joint_xyz="${felis_spool_joint4_xyz}" />
 <!-- Legs -->
 <xacro:quadleg suffix="left" portion="front" geom_rpy="${felis_linkA_joint1_rpy}" joint_xyz="${felis_linkA_joint1_xyz}" />
