Commit message: felis link d

File: defs/robots/felis/felis.common.urdf.xacro (robot description, xacro)
@@ -5,5 +5,5 @@
 <!-- Leg Spool -->
 <xacro:macro name="spool" params="suffix portion geom_rpy joint_xyz">
-	<xacro:urdf_link _name="${suffix}_${portion}_spool_link" _xyz="${felis_spool_xyz}" _rpy="0 0 0"
+	<xacro:urdf_link _name="${suffix}_${portion}_spool_link" _xyz="0 0 0" _rpy="0 0 0"
 		_mesh="${felis_spool_mesh}" _mass="${felis_spool_mass}" _cg="${felis_spool_cg}"
 		_ixx="${felis_spool_ixx}" _iyy="${felis_spool_iyy}" _izz="${felis_spool_izz}"
@@ -13,20 +13,64 @@
 		_upper="${spool_upper_angle}" _effort="${spool_joint_effort}" _velocity="${spool_joint_velocity}" />
 </xacro:macro>
-<!-- Leg Link -->
-<xacro:macro name="quadleg" params="suffix portion geom_rpy joint_xyz">
-	<xacro:urdf_link _name="${suffix}_${portion}_quadleg_linkA" _xyz="${felis_linkA_xyz}" _rpy="0 0 0"
+<!-- Leg Links -->
+<xacro:macro name="quadleg_left" params="portion geom_rpy joint_xyz">
+	<xacro:urdf_link _name="left_${portion}_quadleg_linkA" _xyz="0 0 0" _rpy="0 0 0"
 		_mesh="${felis_linkA_mesh}" _mass="${felis_linkA_mass}" _cg="${felis_linkA_cg}"
 		_ixx="${felis_linkA_ixx}" _iyy="${felis_linkA_iyy}" _izz="${felis_linkA_izz}"
 		_ixy="${felis_linkA_ixy}" _ixz="${felis_linkA_ixz}" _iyz="${felis_linkA_iyz}" />
-	<xacro:urdf_link _name="${suffix}_${portion}_quadleg_linkB" _xyz="${felis_linkB_xyz}" _rpy="${felis_linkB_rpy}"
+	<xacro:urdf_link _name="left_${portion}_quadleg_linkB" _xyz="0 0 0" _rpy="0 0 0"
 		_mesh="${felis_linkB_mesh}" _mass="${felis_linkB_mass}" _cg="${felis_linkB_cg}"
 		_ixx="${felis_linkB_ixx}" _iyy="${felis_linkB_iyy}" _izz="${felis_linkB_izz}"
 		_ixy="${felis_linkB_ixy}" _ixz="${felis_linkB_ixz}" _iyz="${felis_linkB_iyz}" />
-	<xacro:urdf_revolute_joint _name="${suffix}_${portion}_linkA_joint" _parent="base_link"
-		_child="${suffix}_${portion}_quadleg_linkA" _axis="0 1 0" _xyz="${joint_xyz}" _rpy="${geom_rpy}" _lower="${quadleg_jointA_lower_angle}"
+	<xacro:urdf_link _name="left_${portion}_quadleg_linkC" _xyz="0 0 0" _rpy="0 0 0"
+		_mesh="${felis_linkC_mesh}" _mass="${felis_linkC_mass}" _cg="${felis_linkC_cg}"
+		_ixx="${felis_linkC_ixx}" _iyy="${felis_linkC_iyy}" _izz="${felis_linkC_izz}"
+		_ixy="${felis_linkC_ixy}" _ixz="${felis_linkC_ixz}" _iyz="${felis_linkC_iyz}" />
+	<xacro:urdf_link _name="left_${portion}_quadleg_linkD" _xyz="0 0 0" _rpy="0 0 0"
+		_mesh="${felis_linkD_mesh}" _mass="${felis_linkD_mass}" _cg="${felis_linkD_cg}"
+		_ixx="${felis_linkD_ixx}" _iyy="${felis_linkD_iyy}" _izz="${felis_linkD_izz}"
+		_ixy="${felis_linkD_ixy}" _ixz="${felis_linkD_ixz}" _iyz="${felis_linkD_iyz}" />
+	<xacro:urdf_revolute_joint _name="left_${portion}_linkA_joint" _parent="base_link"
+		_child="left_${portion}_quadleg_linkA" _axis="0 0 1" _xyz="${joint_xyz}" _rpy="${geom_rpy}" _lower="${quadleg_jointA_lower_angle}"
 		_upper="${quadleg_jointA_upper_angle}" _effort="${quadleg_joint_effort}" _velocity="${quadleg_joint_velocity}" />
-	<xacro:urdf_revolute_joint _name="${suffix}_${portion}_linkB_joint" _parent="${suffix}_${portion}_quadleg_linkA"
-		_child="${suffix}_${portion}_quadleg_linkB" _axis="0 1 0" _xyz="${felis_linkB_joint_xyz}" _rpy="0 0 0" _lower="${quadleg_jointB_lower_angle}"
+	<xacro:urdf_revolute_joint _name="left_${portion}_linkB_joint" _parent="left_${portion}_quadleg_linkA"
+		_child="left_${portion}_quadleg_linkB" _axis="0 0 1" _xyz="0 0 ${felis_jointAB_zoffset}" _rpy="0 0 -${felis_linkB_starting_angle}" _lower="${quadleg_jointB_lower_angle}"
 		_upper="${quadleg_jointB_upper_angle}" _effort="${quadleg_joint_effort}" _velocity="${quadleg_joint_velocity}" />
+	<xacro:urdf_revolute_joint _name="left_${portion}_linkC_joint" _parent="left_${portion}_quadleg_linkB"
+		_child="left_${portion}_quadleg_linkC" _axis="0 0 1" _xyz="${felis_fulllink_centerlength/2} 0 0" _rpy="0 0 0" _lower="${quadleg_jointC_lower_angle}"
+		_upper="${quadleg_jointC_upper_angle}" _effort="${quadleg_joint_effort}" _velocity="${quadleg_joint_velocity}" />
+	<xacro:urdf_revolute_joint _name="left_${portion}_linkD_joint" _parent="left_${portion}_quadleg_linkC"
+		_child="left_${portion}_quadleg_linkD" _axis="0 0 1" _xyz="${felis_fulllink_centerlength} 0 0" _rpy="0 0 0" _lower="${quadleg_jointD_lower_angle}"
+		_upper="${quadleg_jointD_upper_angle}" _effort="${quadleg_joint_effort}" _velocity="${quadleg_joint_velocity}" />
+</xacro:macro>
+<xacro:macro name="quadleg_right" params="portion geom_rpy joint_xyz">
+	<xacro:urdf_link _name="right_${portion}_quadleg_linkA" _xyz="0 0 0" _rpy="0 ${angle_180d} ${angle_180d}"
+		_mesh="${felis_linkA_mesh}" _mass="${felis_linkA_mass}" _cg="${felis_linkA_cg}"
+		_ixx="${felis_linkA_ixx}" _iyy="${felis_linkA_iyy}" _izz="${felis_linkA_izz}"
+		_ixy="${felis_linkA_ixy}" _ixz="${felis_linkA_ixz}" _iyz="${felis_linkA_iyz}" />
+	<xacro:urdf_link _name="right_${portion}_quadleg_linkB" _xyz="0 0 0" _rpy="0 0 0"
+		_mesh="${felis_linkB_mesh}" _mass="${felis_linkB_mass}" _cg="${felis_linkB_cg}"
+		_ixx="${felis_linkB_ixx}" _iyy="${felis_linkB_iyy}" _izz="${felis_linkB_izz}"
+		_ixy="${felis_linkB_ixy}" _ixz="${felis_linkB_ixz}" _iyz="${felis_linkB_iyz}" />
+	<xacro:urdf_link _name="right_${portion}_quadleg_linkC" _xyz="0 0 0" _rpy="0 ${angle_180d} ${angle_180d}"
+		_mesh="${felis_linkC_mesh}" _mass="${felis_linkC_mass}" _cg="${felis_linkC_cg}"
+		_ixx="${felis_linkC_ixx}" _iyy="${felis_linkC_iyy}" _izz="${felis_linkC_izz}"
+		_ixy="${felis_linkC_ixy}" _ixz="${felis_linkC_ixz}" _iyz="${felis_linkC_iyz}" />
+	<xacro:urdf_link _name="right_${portion}_quadleg_linkD" _xyz="0 0 0" _rpy="0 0 0"
+		_mesh="${felis_linkD_mesh}" _mass="${felis_linkD_mass}" _cg="${felis_linkD_cg}"
+		_ixx="${felis_linkD_ixx}" _iyy="${felis_linkD_iyy}" _izz="${felis_linkD_izz}"
+		_ixy="${felis_linkD_ixy}" _ixz="${felis_linkD_ixz}" _iyz="${felis_linkD_iyz}" />
+	<xacro:urdf_revolute_joint _name="right_${portion}_linkA_joint" _parent="base_link"
+		_child="right_${portion}_quadleg_linkA" _axis="0 0 1" _xyz="${joint_xyz}" _rpy="${geom_rpy}" _lower="${quadleg_jointA_lower_angle}"
+		_upper="${quadleg_jointA_upper_angle}" _effort="${quadleg_joint_effort}" _velocity="${quadleg_joint_velocity}" />
+	<xacro:urdf_revolute_joint _name="right_${portion}_linkB_joint" _parent="right_${portion}_quadleg_linkA"
+		_child="right_${portion}_quadleg_linkB" _axis="0 0 1" _xyz="0 0 ${-felis_jointAB_zoffset-felis_link_width}" _rpy="0 0 -${felis_linkB_starting_angle}" _lower="${quadleg_jointB_lower_angle}"
+		_upper="${quadleg_jointB_upper_angle}" _effort="${quadleg_joint_effort}" _velocity="${quadleg_joint_velocity}" />
+	<xacro:urdf_revolute_joint _name="right_${portion}_linkC_joint" _parent="right_${portion}_quadleg_linkB"
+		_child="right_${portion}_quadleg_linkC" _axis="0 0 1" _xyz="${felis_fulllink_centerlength/2} 0 ${felis_link_width}" _rpy="0 0 0" _lower="${quadleg_jointC_lower_angle}"
+		_upper="${quadleg_jointC_upper_angle}" _effort="${quadleg_joint_effort}" _velocity="${quadleg_joint_velocity}" />
+	<xacro:urdf_revolute_joint _name="right_${portion}_linkD_joint" _parent="right_${portion}_quadleg_linkC"
+		_child="right_${portion}_quadleg_linkD" _axis="0 0 1" _xyz="${felis_fulllink_centerlength} 0 -${felis_link_width}" _rpy="0 0 0" _lower="${quadleg_jointD_lower_angle}"
+		_upper="${quadleg_jointD_upper_angle}" _effort="${quadleg_joint_effort}" _velocity="${quadleg_joint_velocity}" />
 </xacro:macro>
 </robot>

File: defs/robots/felis/felis.common.xacro (robot description, xacro)
@@ -10,52 +10,44 @@
 <xacro:property name="felis_linkE_mesh" value="models/robots/felis/felislinkE.dae" />
 <xacro:property name="felis_linkF_mesh" value="models/robots/felis/felislinkF.dae" />
+<!-- Important Variables -->
+<xacro:property name="felis_z" value="0" />
+<xacro:property name="felis_leg_z" value="0.00990" />
+<xacro:property name="felis_spool_z" value="0.02956" />
+<xacro:property name="felis_jointfront_y" value="0.06030" />
+<xacro:property name="felis_jointrear_y" value="0.06840" />
+<xacro:property name="felis_jointfront_x" value="0.04382" />
+<xacro:property name="felis_jointrear_x" value="0.10099" />
+<xacro:property name="felis_motor_flipdifference" value="0.0202" />
+<xacro:property name="felis_jointAB_zoffset" value="0.004" />
+<xacro:property name="felis_fulllink_centerlength" value="0.07" />
+<xacro:property name="felis_link_width" value="0.006" />
 <!-- Base/Cage Data -->
-<xacro:property name="felis_z" value="0" />
 <xacro:property name="felis_xyz" value="0 0 ${felis_z}" />
 <xacro:property name="felis_rpy" value="0 0 0" />
-<xacro:property name="felis_baselink_cg" value="0 0 0" />
 <!-- Spool Data -->
-<xacro:property name="felis_spool_xyz" value="0 0 0" />
-<xacro:property name="felis_spool_cg" value="0 0 0" />
-<xacro:property name="felis_spool_joint1_xyz" value="0.04382 0.06030 0.02956" />
-<xacro:property name="felis_spool_joint1_rpy" value="-1.570796327 0 0" />
-<xacro:property name="felis_spool_joint2_xyz" value="0.04382 -0.06030 0.02956" />
-<xacro:property name="felis_spool_joint2_rpy" value="1.570796327 -1.570796327 0" />
-<xacro:property name="felis_spool_joint3_xyz" value="-0.12118 0.06840 0.02956" />
-<xacro:property name="felis_spool_joint3_rpy" value="-1.570796327 0 0" />
-<xacro:property name="felis_spool_joint4_xyz" value="-0.12118 -0.06840 0.02956" />
-<xacro:property name="felis_spool_joint4_rpy" value="1.570796327 -1.570796327 0" />
+<xacro:property name="felis_spool_joint_lf_xyz" value="${felis_jointfront_x} ${felis_jointfront_y} ${felis_spool_z}" />
+<xacro:property name="felis_spool_joint_lf_rpy" value="-${angle_90d} 0 0" />
+<xacro:property name="felis_spool_joint_rf_xyz" value="${felis_jointfront_x} -${felis_jointfront_y} ${felis_spool_z}" />
+<xacro:property name="felis_spool_joint_rf_rpy" value="${angle_90d} -${angle_90d} 0" />
+<xacro:property name="felis_spool_joint_lr_xyz" value="-${felis_jointrear_x+felis_motor_flipdifference} ${felis_jointrear_y} ${felis_spool_z}" />
+<xacro:property name="felis_spool_joint_lr_rpy" value="-${angle_90d} 0 0" />
+<xacro:property name="felis_spool_joint_rr_xyz" value="-${felis_jointrear_x+felis_motor_flipdifference} -${felis_jointrear_y} ${felis_spool_z}" />
+<xacro:property name="felis_spool_joint_rr_rpy" value="${angle_90d} -${angle_90d} 0" />
 <!-- Link A Data -->
-<xacro:property name="felis_linkA_xyz" value="0 0 0" />
-<xacro:property name="felis_linkA_cg" value="0 0 0" />
-<xacro:property name="felis_linkA_joint1_xyz" value="0.06401 0.06030 0.00990" />
-<xacro:property name="felis_linkA_joint1_rpy" value="-1.570796327 2.35619449 0" />
-<xacro:property name="felis_linkA_joint2_xyz" value="0 1 0" />
-<xacro:property name="felis_linkA_joint2_rpy" value="0 3.14159 3.14159" />
-<xacro:property name="felis_linkA_joint3_xyz" value="0 1 0" />
-<xacro:property name="felis_linkA_joint3_rpy" value="0 3.14159 3.14159" />
-<xacro:property name="felis_linkA_joint4_xyz" value="0 1 0" />
-<xacro:property name="felis_linkA_joint4_rpy" value="0 3.14159 3.14159" />
+<xacro:property name="felis_linkA_starting_angle" value="${angle_180d-angle_15d}" />
+<xacro:property name="felis_linkA_joint_lf_xyz" value="${felis_jointfront_x+felis_motor_flipdifference} ${felis_jointfront_y} ${felis_leg_z}" />
+<xacro:property name="felis_linkA_joint_rf_xyz" value="${felis_jointfront_x+felis_motor_flipdifference} -${felis_jointfront_y} ${felis_leg_z}" />
+<xacro:property name="felis_linkA_joint_lr_xyz" value="-${felis_jointrear_x} ${felis_jointrear_y} ${felis_leg_z}" />
+<xacro:property name="felis_linkA_joint_rr_xyz" value="-${felis_jointrear_x} -${felis_jointrear_y} ${felis_leg_z}" />
+<xacro:property name="felis_linkA_joint_lf_rpy" value="-${angle_90d} ${felis_linkA_starting_angle} 0" />
+<xacro:property name="felis_linkA_joint_rf_rpy" value="-${angle_90d} ${felis_linkA_starting_angle} 0" />
+<xacro:property name="felis_linkA_joint_lr_rpy" value="-${angle_90d} ${felis_linkA_starting_angle} 0" />
+<xacro:property name="felis_linkA_joint_rr_rpy" value="-${angle_90d} ${felis_linkA_starting_angle} 0" />
 <!-- Link B Data -->
-<xacro:property name="felis_linkB_xyz" value="0 0 0" />
-<xacro:property name="felis_linkB_rpy" value="0 0 0" />
-<xacro:property name="felis_linkB_cg" value="0 0 0" />
-<xacro:property name="felis_linkB_joint_xyz" value="1.5 0 0" />
+<xacro:property name="felis_linkB_starting_angle" value="${angle_180d-angle_30d}" />
 <!-- Link C Data -->
-<xacro:property name="felis_linkC_xyz" value="0 0 0" />
-<xacro:property name="felis_linkC_rpy" value="0 0 0" />
-<xacro:property name="felis_linkC_cg" value="0 0 0" />
 <!-- Link D Data -->
-<xacro:property name="felis_linkD_xyz" value="0 0 0" />
-<xacro:property name="felis_linkD_rpy" value="0 0 0" />
-<xacro:property name="felis_linkD_cg" value="0 0 0" />
 <!-- Link E Data -->
-<xacro:property name="felis_linkE_xyz" value="0 0 0" />
-<xacro:property name="felis_linkE_rpy" value="0 0 0" />
-<xacro:property name="felis_linkE_cg" value="0 0 0" />
 <!-- Link F Data -->
-<xacro:property name="felis_linkF_xyz" value="0 0 0" />
-<xacro:property name="felis_linkF_rpy" value="0 0 0" />
-<xacro:property name="felis_linkF_cg" value="0 0 0" />
 <!-- Joints Constraints -->
 <xacro:property name="spool_lower_angle" value="0" />
@@ -65,4 +57,8 @@
 <xacro:property name="quadleg_jointB_lower_angle"  value="0.0" />
 <xacro:property name="quadleg_jointB_upper_angle"  value="1.4" />
+<xacro:property name="quadleg_jointC_lower_angle"  value="0.0" />
+<xacro:property name="quadleg_jointC_upper_angle"  value="1.4" />
+<xacro:property name="quadleg_jointD_lower_angle"  value="0.0" />
+<xacro:property name="quadleg_jointD_upper_angle"  value="1.4" />
 <!-- Mass -->
 <xacro:property name="felis_baselink_mass" value="1.5" />
@@ -74,4 +70,13 @@
 <xacro:property name="felis_linkE_mass" value="0.2" />
 <xacro:property name="felis_linkF_mass" value="0.2" />
+<!-- Cgs -->
+<xacro:property name="felis_baselink_cg" value="0 0 0" />
+<xacro:property name="felis_spool_cg" value="0 0 0" />
+<xacro:property name="felis_linkA_cg" value="0 0 0" />
+<xacro:property name="felis_linkB_cg" value="0 0 0" />
+<xacro:property name="felis_linkC_cg" value="0 0 0" />
+<xacro:property name="felis_linkD_cg" value="0 0 0" />
+<xacro:property name="felis_linkE_cg" value="0 0 0" />
+<xacro:property name="felis_linkF_cg" value="0 0 0" />
 <!-- Inertial parameters -->
 <xacro:property name="felis_baselink_ixx" value="0.1" />
@@ -131,3 +136,12 @@
 <xacro:property name="quadleg_joint_velocity" value="50" />
 <!-- SDF Specific parameters -->
+<!-- Important Constants -->
+<xacro:property name="angle_05d" value="0.087266463" />
+<xacro:property name="angle_10d" value="0.174532925" />
+<xacro:property name="angle_15d" value="0.261799388" />
+<xacro:property name="angle_30d" value="0.523598776" />
+<xacro:property name="angle_45d" value="0.785398163" />
+<xacro:property name="angle_90d" value="1.570796327" />
+<xacro:property name="angle_135d" value="2.35619449" />
+<xacro:property name="angle_180d" value="3.141592654" />
 </robot>

File: defs/robots/felis/felis.urdf.xacro (robot description, xacro)
@@ -8,9 +8,12 @@
 	_ixy="${felis_baselink_ixy}" _ixz="${felis_baselink_ixz}" _iyz="${felis_baselink_iyz}"/>
 <!-- Spools -->
-<xacro:spool suffix="left" portion="front" geom_rpy="${felis_spool_joint1_rpy}" joint_xyz="${felis_spool_joint1_xyz}" />
-<xacro:spool suffix="right" portion="front" geom_rpy="${felis_spool_joint2_rpy}" joint_xyz="${felis_spool_joint2_xyz}" />
-<xacro:spool suffix="left" portion="rear" geom_rpy="${felis_spool_joint3_rpy}" joint_xyz="${felis_spool_joint3_xyz}" />
-<xacro:spool suffix="right" portion="rear" geom_rpy="${felis_spool_joint4_rpy}" joint_xyz="${felis_spool_joint4_xyz}" />
+<xacro:spool suffix="left" portion="front" geom_rpy="${felis_spool_joint_lf_rpy}" joint_xyz="${felis_spool_joint_lf_xyz}" />
+<xacro:spool suffix="right" portion="front" geom_rpy="${felis_spool_joint_rf_rpy}" joint_xyz="${felis_spool_joint_rf_xyz}" />
+<xacro:spool suffix="left" portion="rear" geom_rpy="${felis_spool_joint_lr_rpy}" joint_xyz="${felis_spool_joint_lr_xyz}" />
+<xacro:spool suffix="right" portion="rear" geom_rpy="${felis_spool_joint_rr_rpy}" joint_xyz="${felis_spool_joint_rr_xyz}" />
 <!-- Legs -->
-<xacro:quadleg suffix="left" portion="front" geom_rpy="${felis_linkA_joint1_rpy}" joint_xyz="${felis_linkA_joint1_xyz}" />
+<xacro:quadleg_left portion="front" geom_rpy="${felis_linkA_joint_lf_rpy}" joint_xyz="${felis_linkA_joint_lf_xyz}" />
+<xacro:quadleg_left portion="rear" geom_rpy="${felis_linkA_joint_lr_rpy}" joint_xyz="${felis_linkA_joint_lr_xyz}" />
+<xacro:quadleg_right portion="front" geom_rpy="${felis_linkA_joint_rf_rpy}" joint_xyz="${felis_linkA_joint_rf_xyz}" />
+<xacro:quadleg_right portion="rear" geom_rpy="${felis_linkA_joint_rr_rpy}" joint_xyz="${felis_linkA_joint_rr_xyz}" />
 </robot>

Commit message: all links felis urdf

File: defs/robots/felis/felis.common.urdf.xacro (robot description, xacro)
@@ -31,4 +31,12 @@
 		_ixx="${felis_linkD_ixx}" _iyy="${felis_linkD_iyy}" _izz="${felis_linkD_izz}"
 		_ixy="${felis_linkD_ixy}" _ixz="${felis_linkD_ixz}" _iyz="${felis_linkD_iyz}" />
+	<xacro:urdf_link _name="left_${portion}_quadleg_linkE" _xyz="0 0 0" _rpy="0 0 0"
+		_mesh="${felis_linkE_mesh}" _mass="${felis_linkE_mass}" _cg="${felis_linkE_cg}"
+		_ixx="${felis_linkE_ixx}" _iyy="${felis_linkE_iyy}" _izz="${felis_linkE_izz}"
+		_ixy="${felis_linkE_ixy}" _ixz="${felis_linkE_ixz}" _iyz="${felis_linkE_iyz}" />
+	<xacro:urdf_link _name="left_${portion}_quadleg_linkF" _xyz="0 0 0" _rpy="0 0 0"
+		_mesh="${felis_linkF_mesh}" _mass="${felis_linkF_mass}" _cg="${felis_linkF_cg}"
+		_ixx="${felis_linkF_ixx}" _iyy="${felis_linkF_iyy}" _izz="${felis_linkF_izz}"
+		_ixy="${felis_linkF_ixy}" _ixz="${felis_linkF_ixz}" _iyz="${felis_linkF_iyz}" />
 	<xacro:urdf_revolute_joint _name="left_${portion}_linkA_joint" _parent="base_link"
 		_child="left_${portion}_quadleg_linkA" _axis="0 0 1" _xyz="${joint_xyz}" _rpy="${geom_rpy}" _lower="${quadleg_jointA_lower_angle}"
@@ -43,4 +51,10 @@
 		_child="left_${portion}_quadleg_linkD" _axis="0 0 1" _xyz="${felis_fulllink_centerlength} 0 0" _rpy="0 0 0" _lower="${quadleg_jointD_lower_angle}"
 		_upper="${quadleg_jointD_upper_angle}" _effort="${quadleg_joint_effort}" _velocity="${quadleg_joint_velocity}" />
+	<xacro:urdf_revolute_joint _name="left_${portion}_linkE_joint" _parent="left_${portion}_quadleg_linkA"
+		_child="left_${portion}_quadleg_linkE" _axis="0 0 1" _xyz="${felis_fulllink_centerlength/2} 0 ${felis_jointAB_zoffset}" _rpy="0 0 0" _lower="${quadleg_jointE_lower_angle}"
+		_upper="${quadleg_jointE_upper_angle}" _effort="${quadleg_joint_effort}" _velocity="${quadleg_joint_velocity}" />
+	<xacro:urdf_revolute_joint _name="left_${portion}_linkF_joint" _parent="left_${portion}_quadleg_linkE"
+		_child="left_${portion}_quadleg_linkF" _axis="0 0 1" _xyz="${felis_fulllink_centerlength} 0 0" _rpy="0 0 0" _lower="${quadleg_jointF_lower_angle}"
+		_upper="${quadleg_jointF_upper_angle}" _effort="${quadleg_joint_effort}" _velocity="${quadleg_joint_velocity}" />
 </xacro:macro>
 <xacro:macro name="quadleg_right" params="portion geom_rpy joint_xyz">
@@ -61,4 +75,12 @@
 		_ixx="${felis_linkD_ixx}" _iyy="${felis_linkD_iyy}" _izz="${felis_linkD_izz}"
 		_ixy="${felis_linkD_ixy}" _ixz="${felis_linkD_ixz}" _iyz="${felis_linkD_iyz}" />
+	<xacro:urdf_link _name="right_${portion}_quadleg_linkE" _xyz="0 0 0" _rpy="0 ${angle_180d} ${angle_180d}"
+		_mesh="${felis_linkE_mesh}" _mass="${felis_linkE_mass}" _cg="${felis_linkE_cg}"
+		_ixx="${felis_linkE_ixx}" _iyy="${felis_linkE_iyy}" _izz="${felis_linkE_izz}"
+		_ixy="${felis_linkE_ixy}" _ixz="${felis_linkE_ixz}" _iyz="${felis_linkE_iyz}" />
+	<xacro:urdf_link _name="right_${portion}_quadleg_linkF" _xyz="0 0 0" _rpy="0 ${angle_180d} ${angle_180d}"
+		_mesh="${felis_linkF_mesh}" _mass="${felis_linkF_mass}" _cg="${felis_linkF_cg}"
+		_ixx="${felis_linkF_ixx}" _iyy="${felis_linkF_iyy}" _izz="${felis_linkF_izz}"
+		_ixy="${felis_linkF_ixy}" _ixz="${felis_linkF_ixz}" _iyz="${felis_linkF_iyz}" />
 	<xacro:urdf_revolute_joint _name="right_${portion}_linkA_joint" _parent="base_link"
 		_child="right_${portion}_quadleg_linkA" _axis="0 0 1" _xyz="${joint_xyz}" _rpy="${geom_rpy}" _lower="${quadleg_jointA_lower_angle}"
@@ -73,4 +95,10 @@
 		_child="right_${portion}_quadleg_linkD" _axis="0 0 1" _xyz="${felis_fulllink_centerlength} 0 -${felis_link_width}" _rpy="0 0 0" _lower="${quadleg_jointD_lower_angle}"
 		_upper="${quadleg_jointD_upper_angle}" _effort="${quadleg_joint_effort}" _velocity="${quadleg_joint_velocity}" />
+	<xacro:urdf_revolute_joint _name="right_${portion}_linkE_joint" _parent="right_${portion}_quadleg_linkA"
+		_child="right_${portion}_quadleg_linkE" _axis="0 0 1" _xyz="${felis_fulllink_centerlength/2} 0 -${felis_jointAB_zoffset}" _rpy="0 0 0" _lower="${quadleg_jointE_lower_angle}"
+		_upper="${quadleg_jointE_upper_angle}" _effort="${quadleg_joint_effort}" _velocity="${quadleg_joint_velocity}" />
+	<xacro:urdf_revolute_joint _name="right_${portion}_linkF_joint" _parent="right_${portion}_quadleg_linkE"
+		_child="right_${portion}_quadleg_linkF" _axis="0 0 1" _xyz="${felis_fulllink_centerlength} 0 0" _rpy="0 0 0" _lower="${quadleg_jointF_lower_angle}"
+		_upper="${quadleg_jointF_upper_angle}" _effort="${quadleg_joint_effort}" _velocity="${quadleg_joint_velocity}" />
 </xacro:macro>
 </robot>

File: defs/robots/felis/felis.common.xacro (robot description, xacro)
@@ -61,4 +61,8 @@
 <xacro:property name="quadleg_jointD_lower_angle"  value="0.0" />
 <xacro:property name="quadleg_jointD_upper_angle"  value="1.4" />
+<xacro:property name="quadleg_jointE_lower_angle"  value="0.0" />
+<xacro:property name="quadleg_jointE_upper_angle"  value="1.4" />
+<xacro:property name="quadleg_jointF_lower_angle"  value="0.0" />
+<xacro:property name="quadleg_jointF_upper_angle"  value="1.4" />
 <!-- Mass -->
 <xacro:property name="felis_baselink_mass" value="1.5" />
