Commit message: modified felis urdf for starting angles

File: defs/robots/felis/felis.common.urdf.xacro (robot description, xacro)
@@ -43,5 +43,5 @@
 		_upper="${quadleg_jointA_upper_angle}" _effort="${quadleg_joint_effort}" _velocity="${quadleg_joint_velocity}" />
 	<xacro:urdf_revolute_joint _name="left_${portion}_linkB_joint" _parent="left_${portion}_quadleg_linkA"
-		_child="left_${portion}_quadleg_linkB" _axis="0 0 1" _xyz="0 0 ${felis_jointAB_zoffset}" _rpy="0 0 -${felis_linkB_starting_angle}" _lower="${quadleg_jointB_lower_angle}"
+		_child="left_${portion}_quadleg_linkB" _axis="0 0 1" _xyz="0 0 ${felis_jointAB_zoffset}" _rpy="0 0 -${felis_linkB_starting_angle_urdf}" _lower="${quadleg_jointB_lower_angle}"
 		_upper="${quadleg_jointB_upper_angle}" _effort="${quadleg_joint_effort}" _velocity="${quadleg_joint_velocity}" />
 	<xacro:urdf_revolute_joint _name="left_${portion}_linkC_joint" _parent="left_${portion}_quadleg_linkB"
@@ -87,5 +87,5 @@
 		_upper="${quadleg_jointA_upper_angle}" _effort="${quadleg_joint_effort}" _velocity="${quadleg_joint_velocity}" />
 	<xacro:urdf_revolute_joint _name="right_${portion}_linkB_joint" _parent="right_${portion}_quadleg_linkA"
-		_child="right_${portion}_quadleg_linkB" _axis="0 0 1" _xyz="0 0 ${-felis_jointAB_zoffset-felis_link_width}" _rpy="0 0 -${felis_linkB_starting_angle}" _lower="${quadleg_jointB_lower_angle}"
+		_child="right_${portion}_quadleg_linkB" _axis="0 0 1" _xyz="0 0 ${-felis_jointAB_zoffset-felis_link_width}" _rpy="0 0 -${felis_linkB_starting_angle_urdf}" _lower="${quadleg_jointB_lower_angle}"
 		_upper="${quadleg_jointB_upper_angle}" _effort="${quadleg_joint_effort}" _velocity="${quadleg_joint_velocity}" />
 	<xacro:urdf_revolute_joint _name="right_${portion}_linkC_joint" _parent="right_${portion}_quadleg_linkB"

File: defs/robots/felis/felis.common.xacro (robot description, xacro)
@@ -38,4 +38,5 @@
 <!-- Link A Data -->
 <xacro:property name="felis_linkA_starting_angle" value="${angle_180d-angle_30d}" />
+<xacro:property name="felis_linkA_starting_angle_urdf" value="0" />
 <!-- Link A Component Wise -->
 <xacro:property name="felis_linkA_joint_lf_x" value="${felis_jointfront_x+felis_motor_flipdifference}" />
@@ -56,10 +57,11 @@
 <xacro:property name="felis_linkA_joint_lr_xyz" value="${felis_linkA_joint_lr_x} ${felis_linkA_joint_lr_y} ${felis_linkA_joint_all_z}" />
 <xacro:property name="felis_linkA_joint_rr_xyz" value="${felis_linkA_joint_rr_x} ${felis_linkA_joint_rr_y} ${felis_linkA_joint_all_z}" />
-<xacro:property name="felis_linkA_joint_lf_rpy" value="${felis_linkA_joint_allrpy_r} ${felis_linkA_joint_allrpy_p} ${felis_linkA_joint_allrpy_y}" />
-<xacro:property name="felis_linkA_joint_rf_rpy" value="${felis_linkA_joint_allrpy_r} ${felis_linkA_joint_allrpy_p} ${felis_linkA_joint_allrpy_y}" />
-<xacro:property name="felis_linkA_joint_lr_rpy" value="${felis_linkA_joint_allrpy_r} ${felis_linkA_joint_allrpy_p} ${felis_linkA_joint_allrpy_y}" />
-<xacro:property name="felis_linkA_joint_rr_rpy" value="${felis_linkA_joint_allrpy_r} ${felis_linkA_joint_allrpy_p} ${felis_linkA_joint_allrpy_y}" />
+<xacro:property name="felis_linkA_joint_lf_rpy" value="${felis_linkA_joint_allrpy_r} ${felis_linkA_starting_angle_urdf} ${felis_linkA_joint_allrpy_y}" />
+<xacro:property name="felis_linkA_joint_rf_rpy" value="${felis_linkA_joint_allrpy_r} ${felis_linkA_starting_angle_urdf} ${felis_linkA_joint_allrpy_y}" />
+<xacro:property name="felis_linkA_joint_lr_rpy" value="${felis_linkA_joint_allrpy_r} ${felis_linkA_starting_angle_urdf} ${felis_linkA_joint_allrpy_y}" />
+<xacro:property name="felis_linkA_joint_rr_rpy" value="${felis_linkA_joint_allrpy_r} ${felis_linkA_starting_angle_urdf} ${felis_linkA_joint_allrpy_y}" />
 <!-- Link B Data -->
 <xacro:property name="felis_linkB_starting_angle" value="${angle_120d}" />
+<xacro:property name="felis_linkB_starting_angle_urdf" value="0" />
 <!-- Link C Data -->
 <!-- Link D Data -->
