Commit message: Added Basic P3AT defs

File: defs/common/common.sdf.xacro (robot description, xacro)
@@ -93,3 +93,10 @@
 	</link>
 </xacro:macro>
+<!-- Macro for color information -->
+<xacro:macro name="gazebo_color" params="color">
+	<material><script>
+		<name>Gazebo/${color}</name>
+		<uri>__default__</uri>
+	</script></material>
+</xacro:macro>
 </sdf>

File: defs/common/common.urdf.xacro (robot description, xacro)
@@ -39,4 +39,21 @@
 			<origin xyz="${_xyz}" rpy="${_rpy}" />
 			<xacro:urdf_mesh _filename="${_mesh}" />
+		</visual>
+		<collision>
+			<origin xyz="${_xyz}" rpy="${_rpy}" />
+			<xacro:urdf_mesh _filename="${_mesh}" />
+		</collision>
+	</link>
+</xacro:macro>
+<xacro:macro name="urdf_link_color" params="_name _xyz _rpy _mesh _mass _cg _ixx _iyy _izz _ixy _ixz _iyz _colorname _rgba">
+	<link name="${_name}">
+		<xacro:urdf_inertial _mass="${_mass}" _cg="${_cg}" _ixx="${_ixx}"
+			_iyy="${_iyy}" _izz="${_izz}" _ixy="${_ixy}" _ixz="${_ixz}" _iyz="${_iyz}" />
+		<visual>
+			<origin xyz="${_xyz}" rpy="${_rpy}" />
+			<xacro:urdf_mesh _filename="${_mesh}" />
+			<material name="${_colorname}">
+				<color rgba="${_rgba}"/>
+			</material>
 		</visual>
 		<collision>

File: defs/robots/risewheelchair/risewheelchair.common.xacro (robot description, xacro)
@@ -38,5 +38,5 @@
 <xacro:property name="caster_axis" value="0 0 1" />
 <!-- Mass and Inertias -->
-<xacro:property name="wheelchair_mass" value="60.0" />
+<xacro:property name="wheelchair_mass" value="80.0" />
 <xacro:property name="wheelchair_sicklms_mass" value="4.5" />
 <xacro:property name="bender_mass" value="70" />

Commit message: Felis left portion without spring

File: defs/common/common.sdf.xacro (robot description, xacro)
@@ -77,4 +77,13 @@
 	<kinematic>0</kinematic>
 </xacro:macro>
+<xacro:macro name="link_def_extra_selfcollide">
+	<velocity_decay>
+		<linear>0.001</linear>
+		<angular>0.001</angular>
+	</velocity_decay>
+	<gravity>1</gravity>
+	<self_collide>1</self_collide>
+	<kinematic>0</kinematic>
+</xacro:macro>
 <!-- Macro for null link in sdf -->
 <xacro:macro name="sdf_link_null" params="_name geom_rpy joint_xyz">

File: defs/robots/felis/felis.common.sdf.xacro (robot description, xacro)
@@ -23,4 +23,121 @@
 				_lower="${spool_lower_angle}" _upper="${spool_upper_angle}" _useparent="0" />
 </xacro:macro>
-<!-- Legs -->
+<!--Left Leg -->
+<xacro:macro name="quadleg_left" params="portion geom_r geom_p geom_y joint_x joint_y joint_z">
+	<link name="left_${portion}_quadleg_linkA">
+		<xacro:link_def_extra_selfcollide />
+		<pose>${joint_x} ${joint_y} ${joint_z} ${geom_r} ${geom_p} ${geom_y}</pose>
+		<xacro:sdf_inertial _mass="${felis_linkA_mass}" _cg="${felis_linkA_cg}"
+				_ixx="${felis_linkA_ixx}" _iyy="${felis_linkA_iyy}" _izz="${felis_linkA_izz}" _ixy="${felis_linkA_ixy}"
+				_ixz="${felis_linkA_ixz}" _iyz="${felis_linkA_iyz}" />
+		<visual name="left_${portion}_quadleg_linkA_visual">
+			<pose>0 0 0 0 0 0</pose>
+			<xacro:sdf_mesh _filename="${felis_linkA_mesh}" />
+		</visual>
+		<collision name="left_${portion}_quadleg_linkA_collision">
+			<pose>0 0 0 0 0 0</pose>
+			<xacro:sdf_mesh _filename="${felis_linkA_mesh}" />
+			<xacro:sdf_collision_params kp="${links_kp}" kd="${links_kd}" mu="${links_mu}" mu2="${links_mu2}"
+				slip1="${links_slip1}" slip2="${links_slip2}" fdir1="${links_fdir1}" max_contacts="${links_max_contacts}"/>
+		</collision>
+	</link>
+	<link name="left_${portion}_quadleg_linkB">
+		<xacro:link_def_extra_selfcollide />
+		<pose >${joint_x} ${joint_y + felis_jointAB_zoffset} ${joint_z} ${geom_r} ${geom_p-felis_linkB_starting_angle} ${geom_y}</pose>
+		<xacro:sdf_inertial _mass="${felis_linkB_mass}" _cg="${felis_linkB_cg}"
+				_ixx="${felis_linkB_ixx}" _iyy="${felis_linkB_iyy}" _izz="${felis_linkB_izz}" _ixy="${felis_linkB_ixy}"
+				_ixz="${felis_linkB_ixz}" _iyz="${felis_linkB_iyz}" />
+		<visual name="left_${portion}_quadleg_linkB_visual">
+			<pose>0 0 0 0 0 0</pose>
+			<xacro:sdf_mesh _filename="${felis_linkB_mesh}" />
+		</visual>
+		<collision name="left_${portion}_quadleg_linkB_collision">
+			<pose>0 0 0 0 0 0</pose>
+			<xacro:sdf_mesh _filename="${felis_linkB_mesh}" />
+			<xacro:sdf_collision_params kp="${links_kp}" kd="${links_kd}" mu="${links_mu}" mu2="${links_mu2}"
+				slip1="${links_slip1}" slip2="${links_slip2}" fdir1="${links_fdir1}" max_contacts="${links_max_contacts}"/>
+		</collision>
+	</link>
+	<link name="left_${portion}_quadleg_linkC">
+		<xacro:link_def_extra_selfcollide />
+		<pose >${joint_x + (felis_fulllink_centerlength/2)} ${joint_y + felis_jointAB_zoffset} ${joint_z} ${geom_r} ${geom_p-felis_linkB_starting_angle} ${geom_y}</pose>
+		<xacro:sdf_inertial _mass="${felis_linkC_mass}" _cg="${felis_linkC_cg}"
+				_ixx="${felis_linkC_ixx}" _iyy="${felis_linkC_iyy}" _izz="${felis_linkC_izz}" _ixy="${felis_linkC_ixy}"
+				_ixz="${felis_linkC_ixz}" _iyz="${felis_linkC_iyz}" />
+		<visual name="left_${portion}_quadleg_linkC_visual">
+			<pose>0 0 0 0 0 0</pose>
+			<xacro:sdf_mesh _filename="${felis_linkC_mesh}" />
+		</visual>
+		<collision name="left_${portion}_quadleg_linkC_collision">
+			<pose>0 0 0 0 0 0</pose>
+			<xacro:sdf_mesh _filename="${felis_linkC_mesh}" />
+			<xacro:sdf_collision_params kp="${links_kp}" kd="${links_kd}" mu="${links_mu}" mu2="${links_mu2}"
+				slip1="${links_slip1}" slip2="${links_slip2}" fdir1="${links_fdir1}" max_contacts="${links_max_contacts}"/>
+		</collision>
+	</link>
+	<link name="left_${portion}_quadleg_linkD">
+		<xacro:link_def_extra_selfcollide />
+		<pose >${joint_x + 3*(felis_fulllink_centerlength/2)} ${joint_y + felis_jointAB_zoffset} ${joint_z} ${geom_r} ${geom_p-felis_linkB_starting_angle} ${geom_y}</pose>
+		<xacro:sdf_inertial _mass="${felis_linkD_mass}" _cg="${felis_linkD_cg}"
+				_ixx="${felis_linkD_ixx}" _iyy="${felis_linkD_iyy}" _izz="${felis_linkD_izz}" _ixy="${felis_linkD_ixy}"
+				_ixz="${felis_linkD_ixz}" _iyz="${felis_linkD_iyz}" />
+		<visual name="left_${portion}_quadleg_linkD_visual">
+			<pose>0 0 0 0 0 0</pose>
+			<xacro:sdf_mesh _filename="${felis_linkD_mesh}" />
+		</visual>
+		<collision name="left_${portion}_quadleg_linkD_collision">
+			<pose>0 0 0 0 0 0</pose>
+			<xacro:sdf_mesh _filename="${felis_linkD_mesh}" />
+			<xacro:sdf_collision_params kp="${links_kp}" kd="${links_kd}" mu="${links_mu}" mu2="${links_mu2}"
+				slip1="${links_slip1}" slip2="${links_slip2}" fdir1="${links_fdir1}" max_contacts="${links_max_contacts}"/>
+		</collision>
+	</link>
+	<link name="left_${portion}_quadleg_linkE">
+		<xacro:link_def_extra_selfcollide />
+		<pose >${joint_x + (felis_fulllink_centerlength/2)} ${joint_y + felis_jointAB_zoffset} ${joint_z} ${geom_r} ${geom_p-felis_linkB_starting_angle} ${geom_y}</pose>
+		<xacro:sdf_inertial _mass="${felis_linkE_mass}" _cg="${felis_linkE_cg}"
+				_ixx="${felis_linkE_ixx}" _iyy="${felis_linkE_iyy}" _izz="${felis_linkE_izz}" _ixy="${felis_linkE_ixy}"
+				_ixz="${felis_linkE_ixz}" _iyz="${felis_linkE_iyz}" />
+		<visual name="left_${portion}_quadleg_linkE_visual">
+			<pose>0 0 0 0 0 0</pose>
+			<xacro:sdf_mesh _filename="${felis_linkE_mesh}" />
+		</visual>
+		<collision name="left_${portion}_quadleg_linkE_collision">
+			<pose>0 0 0 0 0 0</pose>
+			<xacro:sdf_mesh _filename="${felis_linkE_mesh}" />
+			<xacro:sdf_collision_params kp="${links_kp}" kd="${links_kd}" mu="${links_mu}" mu2="${links_mu2}"
+				slip1="${links_slip1}" slip2="${links_slip2}" fdir1="${links_fdir1}" max_contacts="${links_max_contacts}"/>
+		</collision>
+	</link>
+	<link name="left_${portion}_quadleg_linkF">
+		<xacro:link_def_extra_selfcollide />
+		<pose >${joint_x + 3*(felis_fulllink_centerlength/2)} ${joint_y + felis_jointAB_zoffset} ${joint_z} ${geom_r} ${geom_p-felis_linkB_starting_angle} ${geom_y}</pose>
+		<xacro:sdf_inertial _mass="${felis_linkE_mass}" _cg="${felis_linkF_cg}"
+				_ixx="${felis_linkF_ixx}" _iyy="${felis_linkF_iyy}" _izz="${felis_linkF_izz}" _ixy="${felis_linkF_ixy}"
+				_ixz="${felis_linkF_ixz}" _iyz="${felis_linkF_iyz}" />
+		<visual name="left_${portion}_quadleg_linkF_visual">
+			<pose>0 0 0 0 0 0</pose>
+			<xacro:sdf_mesh _filename="${felis_linkF_mesh}" />
+		</visual>
+		<collision name="left_${portion}_quadleg_linkF_collision">
+			<pose>0 0 0 0 0 0</pose>
+			<xacro:sdf_mesh _filename="${felis_linkF_mesh}" />
+			<xacro:sdf_collision_params kp="${links_kp}" kd="${links_kd}" mu="${links_mu}" mu2="${links_mu2}"
+				slip1="${links_slip1}" slip2="${links_slip2}" fdir1="${links_fdir1}" max_contacts="${links_max_contacts}"/>
+		</collision>
+	</link>
+	<xacro:sdf_revolute_joint _name="left_${portion}_linkA_joint" _parent="base_link" _child="left_${portion}_quadleg_linkA" _axis="0 0 1"
+				_lower="${quadleg_jointA_lower_angle}" _upper="${quadleg_jointA_upper_angle}" _useparent="0" />
+	<xacro:sdf_revolute_joint _name="left_${portion}_linkB_joint" _parent="left_${portion}_quadleg_linkA" _child="left_${portion}_quadleg_linkB" _axis="0 0 1"
+				_lower="${quadleg_jointB_lower_angle}" _upper="${quadleg_jointB_upper_angle}" _useparent="0" />
+	<xacro:sdf_revolute_joint _name="left_${portion}_linkC_joint" _parent="left_${portion}_quadleg_linkB" _child="left_${portion}_quadleg_linkC" _axis="0 0 1"
+				_lower="${quadleg_jointC_lower_angle}" _upper="${quadleg_jointC_upper_angle}" _useparent="0" />
+	<xacro:sdf_revolute_joint _name="left_${portion}_linkD_joint" _parent="left_${portion}_quadleg_linkC" _child="left_${portion}_quadleg_linkD" _axis="0 0 1"
+				_lower="${quadleg_jointD_lower_angle}" _upper="${quadleg_jointD_upper_angle}" _useparent="0" />
+	<xacro:sdf_revolute_joint _name="left_${portion}_linkE_joint" _parent="left_${portion}_quadleg_linkA" _child="left_${portion}_quadleg_linkE" _axis="0 0 1"
+				_lower="${quadleg_jointE_lower_angle}" _upper="${quadleg_jointE_upper_angle}" _useparent="0" />
+	<xacro:sdf_revolute_joint _name="left_${portion}_linkF_joint" _parent="left_${portion}_quadleg_linkE" _child="left_${portion}_quadleg_linkF" _axis="0 0 1"
+				_lower="${quadleg_jointF_lower_angle}" _upper="${quadleg_jointF_upper_angle}" _useparent="0" />
+</xacro:macro>
+<!-- Right Leg -->
 </sdf>

File: defs/robots/felis/felis.common.xacro (robot description, xacro)
@@ -38,12 +38,26 @@
 <!-- Link A Data -->
 <xacro:property name="felis_linkA_starting_angle" value="0" />
-<xacro:property name="felis_linkA_joint_lf_xyz" value="${felis_jointfront_x+felis_motor_flipdifference} ${felis_jointfront_y} ${felis_leg_z}" />
-<xacro:property name="felis_linkA_joint_rf_xyz" value="${felis_jointfront_x+felis_motor_flipdifference} -${felis_jointfront_y} ${felis_leg_z}" />
-<xacro:property name="felis_linkA_joint_lr_xyz" value="-${felis_jointrear_x} ${felis_jointrear_y} ${felis_leg_z}" />
-<xacro:property name="felis_linkA_joint_rr_xyz" value="-${felis_jointrear_x} -${felis_jointrear_y} ${felis_leg_z}" />
-<xacro:property name="felis_linkA_joint_lf_rpy" value="-${angle_90d} ${felis_linkA_starting_angle} 0" />
-<xacro:property name="felis_linkA_joint_rf_rpy" value="-${angle_90d} ${felis_linkA_starting_angle} 0" />
-<xacro:property name="felis_linkA_joint_lr_rpy" value="-${angle_90d} ${felis_linkA_starting_angle} 0" />
-<xacro:property name="felis_linkA_joint_rr_rpy" value="-${angle_90d} ${felis_linkA_starting_angle} 0" />
+<!-- Link A Component Wise -->
+<xacro:property name="felis_linkA_joint_lf_x" value="${felis_jointfront_x+felis_motor_flipdifference}" />
+<xacro:property name="felis_linkA_joint_lf_y" value="${felis_jointfront_y}" />
+<xacro:property name="felis_linkA_joint_rf_x" value="${felis_jointfront_x+felis_motor_flipdifference}" />
+<xacro:property name="felis_linkA_joint_rf_y" value="-${felis_jointfront_y}" />
+<xacro:property name="felis_linkA_joint_lr_x" value="-${felis_jointrear_x}" />
+<xacro:property name="felis_linkA_joint_lr_y" value="${felis_jointrear_y}" />
+<xacro:property name="felis_linkA_joint_rr_x" value="-${felis_jointrear_x}" />
+<xacro:property name="felis_linkA_joint_rr_y" value="-${felis_jointrear_y}" />
+<xacro:property name="felis_linkA_joint_all_z" value="${felis_leg_z}" />
+<xacro:property name="felis_linkA_joint_allrpy_r" value="-${angle_90d}" />
+<xacro:property name="felis_linkA_joint_allrpy_p" value="${felis_linkA_starting_angle}" />
+<xacro:property name="felis_linkA_joint_allrpy_y" value="0" />
+<!-- Link A pose vectors -->
+<xacro:property name="felis_linkA_joint_lf_xyz" value="${felis_linkA_joint_lf_x} ${felis_linkA_joint_lf_y} ${felis_linkA_joint_all_z}" />
+<xacro:property name="felis_linkA_joint_rf_xyz" value="${felis_linkA_joint_rf_x} ${felis_linkA_joint_rf_y} ${felis_linkA_joint_all_z}" />
+<xacro:property name="felis_linkA_joint_lr_xyz" value="${felis_linkA_joint_lr_x} ${felis_linkA_joint_lr_y} ${felis_linkA_joint_all_z}" />
+<xacro:property name="felis_linkA_joint_rr_xyz" value="${felis_linkA_joint_rr_x} ${felis_linkA_joint_lf_y} ${felis_linkA_joint_all_z}" />
+<xacro:property name="felis_linkA_joint_lf_rpy" value="${felis_linkA_joint_allrpy_r} ${felis_linkA_joint_allrpy_p} ${felis_linkA_joint_allrpy_y}" />
+<xacro:property name="felis_linkA_joint_rf_rpy" value="${felis_linkA_joint_allrpy_r} ${felis_linkA_joint_allrpy_p} ${felis_linkA_joint_allrpy_y}" />
+<xacro:property name="felis_linkA_joint_lr_rpy" value="${felis_linkA_joint_allrpy_r} ${felis_linkA_joint_allrpy_p} ${felis_linkA_joint_allrpy_y}" />
+<xacro:property name="felis_linkA_joint_rr_rpy" value="${felis_linkA_joint_allrpy_r} ${felis_linkA_joint_allrpy_p} ${felis_linkA_joint_allrpy_y}" />
 <!-- Link B Data -->
 <xacro:property name="felis_linkB_starting_angle" value="0" />
@@ -57,6 +71,6 @@
 <xacro:property name="quadleg_jointA_lower_angle"  value="${angle_60d+angle_15d}" /> <!-- Use Exact Values -->
 <xacro:property name="quadleg_jointA_upper_angle"  value="${angle_180d - angle_15d}" /><!-- Use Exact Values -->
-<xacro:property name="quadleg_jointB_lower_angle"  value="${joint_min_angle}" /><!-- Use Exact Values -->
-<xacro:property name="quadleg_jointB_upper_angle"  value="${joint_max_angle}" /><!-- Use Exact Values -->
+<xacro:property name="quadleg_jointB_lower_angle"  value="-${joint_max_angle}" /><!-- Use Exact Values -->
+<xacro:property name="quadleg_jointB_upper_angle"  value="${joint_min_angle}" /><!-- Use Exact Values -->
 <xacro:property name="quadleg_jointC_lower_angle"  value="${joint_min_angle}" /><!-- Use Exact Values -->
 <xacro:property name="quadleg_jointC_upper_angle"  value="${joint_max_angle}" /><!-- Use Exact Values -->
@@ -141,5 +155,13 @@
 <xacro:property name="quadleg_joint_effort" value="100" />
 <xacro:property name="quadleg_joint_velocity" value="50" />
+<xacro:property name="links_kp" value="1e+06" />
+<xacro:property name="links_kd" value="100" />
+<xacro:property name="links_mu" value="0.3" />
+<xacro:property name="links_mu2" value="0.5" />
+<xacro:property name="links_slip1" value="0.5" />
+<xacro:property name="links_slip2" value="0.2" />
+<xacro:property name="links_fdir1" value="1 0 0" />
 <!-- SDF Specific parameters -->
+<xacro:property name="links_max_contacts" value="6" />
 <!-- Important Constants -->
 <xacro:property name="angle_05d" value="0.087266463" />

File: defs/robots/felis/felis.sdf.xacro (robot description, xacro)
@@ -4,5 +4,5 @@
 	<model name="risewheelchair">
 		<static>0</static>
-		<pose>0 0 0 0 0 0</pose>
+		<pose>0 0 0.082 0 0 0</pose>
 		<!-- Base Link -->
 		<link name="base_link">
@@ -20,4 +20,5 @@
 				<xacro:sdf_mesh _filename="${felis_base_mesh}" />
 			</collision>
+			<must_be_base_link> 1 </must_be_base_link>
 			<!-- Basic Camera TODO-->
 		</link>
@@ -28,4 +29,8 @@
 		<xacro:spool suffix="right" portion="rear" geom_rpy="${felis_spool_joint_rr_rpy}" joint_xyz="${felis_spool_joint_rr_xyz}" />
 		<!-- Legs -->
+		<xacro:quadleg_left portion="front" geom_r="${felis_linkA_joint_allrpy_r}" geom_p="${felis_linkA_joint_allrpy_p}" geom_y="${felis_linkA_joint_allrpy_y}"
+			joint_x="${felis_linkA_joint_lf_x}" joint_y="${felis_linkA_joint_lf_y}" joint_z="${felis_linkA_joint_all_z}" />
+		<xacro:quadleg_left portion="rear" geom_r="${felis_linkA_joint_allrpy_r}" geom_p="${felis_linkA_joint_allrpy_p}" geom_y="${felis_linkA_joint_allrpy_y}"
+			joint_x="${felis_linkA_joint_lr_x}" joint_y="${felis_linkA_joint_lr_y}" joint_z="${felis_linkA_joint_all_z}" />
 	</model>
 </sdf>
